Commit message: the final commit of the project

File: robot_description/urdf/chassis.urdf.xacro (robot description, xacro)
@@ -148,5 +148,4 @@
             <origin xyz="0 0 0" rpy="0 0 0" />
             <geometry>
-                <box size="0.0 0.0 0.0"/>
             </geometry>
         </collision>
@@ -157,4 +156,26 @@
                      iyy="0.329853029043022" iyz="-0.0000005106111186954"
                      izz="0.502514023614247" />
+        </inertial>
+    </link>
+    <link name="lidarbase_link">
+        <visual>
+            <origin xyz="0 0 0" rpy="0 0 0" />
+            <geometry>
+                <mesh filename="package://robot_description/meshes/liDAR_SPACER.STL"/>
+            </geometry>
+            <material name="Orange_body"/>
+        </visual>
+        <collision>
+            <origin xyz="0 0 0" rpy="0 0 0" />
+            <geometry>
+                <box size="0.0 0.0 0.0"/>
+            </geometry>
+        </collision>
+        <inertial>
+            <mass value="0.044971" />
+            <origin xyz="0 0 0" />
+            <inertia ixx="0.000019021" ixy="-1.0558E-020" ixz="-0.0000096066"
+                     iyy="0.000053096" iyz="-6.5811E-021"
+                     izz="0.000065593" />
         </inertial>
     </link>
@@ -194,3 +215,8 @@
         <origin xyz="0.0 0.0 0.2374" rpy="0.0 0.0 0.0"/>
     </joint>
+    <joint name="base_lidarbase_joint" type="fixed">
+        <parent link="base_link"/>
+        <child link="lidarbase_link"/>
+        <origin xyz="0.44615 0.0325 0.026" rpy="0.0 0.0 0.0"/>
+    </joint>
 </robot>

File: robot_description/urdf/ros2_control.urdf.xacro (robot description, xacro)
@@ -1,5 +1,5 @@
 <?xml version="1.0"?>
 <robot xmlns:xacro="http://www.ros.org/wiki/xacro">
-    <!-- <ros2_control name="MPU6050" type="system">
+    <!--<ros2_control name="MPU6050" type="system">
         <hardware>
             <plugin>mpu6050_hardware/Mpu6050HardwareInterface</plugin>
@@ -12,6 +12,10 @@
             <state_interface name="angular_velocity.y"/>
             <state_interface name="angular_velocity.z"/>
+            <state_interface name="orientation.x"/>
+            <state_interface name="orientation.y"/>
+            <state_interface name="orientation.z"/>
+            <state_interface name="orientation.w"/>
         </sensor>
-    </ros2_control> -->
+    </ros2_control>-->
     <ros2_control name="MobileBase" type="system">
         <hardware>

File: robot_description/urdf/sensors.urdf.xacro (robot description, xacro)
@@ -1,20 +1,20 @@
 <?xml version="1.0"?>
 <robot xmlns:xacro="http://www.ros.org/wiki/xacro">
-    <!-- <link name="imu_link">
-        <visual>
-            <origin xyz="0 0 0" rpy="0 0 0" />
-            <geometry>
-                <mesh filename="package://package_name/meshes/mesh.stl" />
-            </geometry>
-            <material name="Blue_tech"/>
-        </visual>
-        <collision>
-            <origin xyz="0 0 0" rpy="0 0 0" />
-            <geometry>
-                <box size="0.0 0.0 0.0"/>
-            </geometry>
-        </collision>
-        <inertial>
-            <mass value="1.0" />
+    <link name="imu_link">
+        <visual>
+            <origin xyz="0 0 0" rpy="0 0 0" />
+            <geometry>
+                <box size="0.03 0.02 0.01"/>
+            </geometry>
+            <material name="Blue_tech"/>
+        </visual>
+        <collision>
+            <origin xyz="0 0 0" rpy="0 0 0" />
+            <geometry>
+                <box size="0.03 0.02 0.01"/>
+            </geometry>
+        </collision>
+        <inertial>
+            <mass value="0.05" />
             <origin xyz="0 0 0" />
             <inertia ixx="1.0" ixy="0.0" ixz="0.0"
@@ -22,5 +22,5 @@
                      izz="1.0" />
         </inertial>
-    </link> -->
+    </link>
     <link name="Camera_link">
         <visual>
@@ -183,5 +183,5 @@
         <parent link="base_link"/>
         <child link="base_laser"/>
-        <origin xyz="0.344 0.0 0.014" rpy="0.0 0.0 0.0"/>
+        <origin xyz="0.412 0.0 0.038" rpy="0.0 0.0 -1.57"/>
     </joint>
     <joint name="base_ultra1_joint" type="fixed">
@@ -210,3 +210,8 @@
         <origin xyz="0.0 0.0 0.00155" rpy="0.0 0.0 0.0"/>
     </joint>
+    <joint name="base_imu_joint" type="fixed">
+        <parent link="base_link"/>
+        <child link="imu_link"/>
+        <origin xyz="0.255 -0.1 0.025" rpy="0.0 0.0 0.0"/>
+    </joint>
 </robot>
